Commit message: The hexa is still not flying using mavproxy

File: urdf/hexacopter.urdf (robot description, URDF)
Before this commit: robot hexacopter, 7 links, 6 joints
Links:
- link Prop_1: geometry collision mesh filename=package://hexacopter_ardupilot/urdf/meshes/Prop_1.STL; visual mesh filename=package://hexacopter_ardupilot/urdf/meshes/Prop_1.STL
- link Prop_2: geometry collision mesh filename=package://hexacopter_ardupilot/urdf/meshes/Prop_2.STL; visual mesh filename=package://hexacopter_ardupilot/urdf/meshes/Prop_2.STL
- link Prop_3: geometry collision mesh filename=package://hexacopter_ardupilot/urdf/meshes/Prop_3.STL; visual mesh filename=package://hexacopter_ardupilot/urdf/meshes/Prop_3.STL
- link Prop_4: geometry collision mesh filename=package://hexacopter_ardupilot/urdf/meshes/Prop_4.STL; visual mesh filename=package://hexacopter_ardupilot/urdf/meshes/Prop_4.STL
- link Prop_5: geometry collision mesh filename=package://hexacopter_ardupilot/urdf/meshes/Prop_5.STL; visual mesh filename=package://hexacopter_ardupilot/urdf/meshes/Prop_5.STL
- link Prop_6: geometry collision mesh filename=package://hexacopter_ardupilot/urdf/meshes/Prop_6.STL; visual mesh filename=package://hexacopter_ardupilot/urdf/meshes/Prop_6.STL
- link base_link: geometry collision mesh filename=package://hexacopter_ardupilot/urdf/meshes/base_link.STL; visual mesh filename=package://hexacopter_ardupilot/urdf/meshes/base_link.STL
